File: PCB/PCB-Badge/PCB-Badge.kicad_pcb (KiCad board)
At the start: 2 copper layers, 71 x 95.6 mm, 5 parts, among them U1 NT3H2111W0FT1X

Commit message: Silkscreen + Gerbers
Parts:
- added G*** (x2): LOGO, Silkscreen:hackclub-square, F.Cu at (187.2, 123.5)
- added G*** (x2): LOGO, Silkscreen:soup, F.Cu at (164.0, 65.7)
- added G***: LOGO, Silkscreen:ZBoard-V1-Logo, B.Cu at (171.7, 71.6)
- added G*** (x2): LOGO, Silkscreen:hackclub-logo, B.Cu at (187.4, 98.0)
- added G***: LOGO, Silkscreen:HexiLux-Logo, B.Cu at (175.7, 67.8)
Other:
- board text added: "(Obviously)"
- board text added: "Fallout!!!"
- board text added: "Hack Clubber"
- board text added: "Jay G"
- board text added: "Made for Hack Club Fallout"
- board text added: "SCAN HERE"
- board text added: "Slack: @ZeusyBoy"
- board text added: "https://github.com/ZeusyBoy98"
